Commit message: replace carlikebot mesh to '1:10 Tesla Model 3'

File: ros2_control_demo_description/carlikebot/urdf/carlikebot_description.urdf.xacro (robot description, xacro)
@@ -4,13 +4,18 @@
   <!-- Constants for robot dimensions -->
   <xacro:property name="PI" value="3.1415926535897931"/>
+  <xacro:property name="mesh_scale" value="0.001 0.001 0.001" /> <!-- from millimeter to meter -->
+  <xacro:property name="mesh_fpath" value="package://ros2_control_demo_description/carlikebot/meshes/tesla_model3_rc_car_body.stl" />
   <xacro:property name="base_mass" value="4.0" /> <!-- arbitrary value for base mass -->
-  <xacro:property name="base_width" value="0.260" />
-  <xacro:property name="base_length" value="0.525" />
-  <xacro:property name="base_height" value="0.060" />
-  <xacro:property name="wheelbase" value="0.325" />
-  <xacro:property name="wheel_mass" value="0.34055" /> <!-- arbitrary value for wheel mass -->
-  <xacro:property name="wheel_len" value="0.045" />
-  <xacro:property name="wheel_radius" value="0.05" />
-  <!-- <xacro:property name="wheeltrack" value="" -->
+  <xacro:property name="base_width" value="0.185" />
+  <xacro:property name="base_length" value="0.423" />
+  <xacro:property name="base_height" value="0.124" />
+  <xacro:property name="base_xoff" value="0.110" /> <!-- x-offset of base to rear-axle center -->
+  <xacro:property name="base_yoff" value="0.000" /> <!-- y-offset of base to rear-axle center -->
+  <xacro:property name="base_zoff" value="0.013" /> <!-- z-offset of base to rear-axle center -->
+  <xacro:property name="wheel_base" value="0.258" />
+  <xacro:property name="wheel_mass" value="0.025" /> <!-- arbitrary value for wheel mass -->
+  <xacro:property name="wheel_width" value="0.023" />
+  <xacro:property name="wheel_radius" value="0.030" />
+  <xacro:property name="wheel_track" value="${base_width-wheel_width}"/>
   <!-- Base Link -->
   <link name="${prefix}base_link" />
@@ -18,15 +23,15 @@
   <link name="${prefix}chassis_link">
     <collision>
-      <origin xyz="0 0 0" rpy="0 0 0"/>
+      <origin xyz="0 0 0" rpy="0 0 ${PI/2}"/>
       <geometry>
-        <box size="${base_length} ${base_width} ${base_height}"/>
+        <mesh filename="${mesh_fpath}" scale="${mesh_scale}"/>
       </geometry>
     </collision>
     <visual>
-      <origin xyz="0 0 0" rpy="0 0 0"/>
+      <origin xyz="0 0 0" rpy="0 0 ${PI/2}"/>
       <geometry>
-        <box size="${base_length} ${base_width} ${base_height}"/>
+        <mesh filename="${mesh_fpath}"  scale="${mesh_scale}"/>
       </geometry>
-      <material name="orange"/>
+      <material name="white"/>
     </visual>
     <inertial>
@@ -42,5 +47,5 @@
       <parent link="${prefix}base_link"/>
       <child link="${prefix}chassis_link"/>
-      <origin xyz="0 0 ${base_height/2 + wheel_radius}" rpy="0 0 0"/>
+      <origin xyz="${base_xoff} ${base_yoff} ${base_zoff - wheel_radius}" rpy="0 0 0"/>
       <axis xyz="0 0 1"/>
       <dynamics damping="0.2"/>
@@ -58,7 +63,7 @@
     </link>
     <joint name="${prefix}virtual_rear_wheel_joint" type="continuous">
-      <parent link="${prefix}chassis_link"/>
+      <parent link="${prefix}base_link"/>
       <child link="${prefix}virtual_rear_wheel"/>
-      <origin xyz="-${wheelbase/2} 0 -${base_height/2}" rpy="0 0 ${PI/2}"/>
+      <origin xyz="0 0 0" rpy="0 0 ${PI/2}"/>
       <axis xyz="1 0 0"/>
       <limit effort="100.0" velocity="100.0"/>
@@ -70,5 +75,5 @@
         <origin xyz="0 0 0" rpy="${PI/2} 0 ${PI/2}"/>
         <geometry>
-          <cylinder length="${wheel_len}" radius="${wheel_radius}"/>
+          <cylinder length="${wheel_width}" radius="${wheel_radius}"/>
         </geometry>
       </collision>
@@ -76,5 +81,5 @@
         <origin xyz="0 0 0" rpy="${PI/2} 0 ${PI/2}"/>
         <geometry>
-          <cylinder length="${wheel_len}" radius="${wheel_radius}"/>
+          <cylinder length="${wheel_width}" radius="${wheel_radius}"/>
         </geometry>
         <material name="black"/>
@@ -90,7 +95,7 @@
     </link>
     <joint name="${prefix}rear_right_wheel_joint" type="continuous">
-      <parent link="${prefix}chassis_link"/>
+      <parent link="${prefix}base_link"/>
       <child link="${prefix}rear_right_wheel"/>
-      <origin xyz="-${wheelbase/2} ${base_width/2} -${base_height/2}" rpy="0 0 ${PI/2}"/>
+      <origin xyz="0 -${wheel_track/2} 0" rpy="0 0 ${PI/2}"/>
       <axis xyz="1 0 0"/>
       <limit effort="100.0" velocity="100.0"/>
@@ -103,5 +108,5 @@
           <origin xyz="0 0 0" rpy="${PI/2} 0 ${PI/2}"/>
           <geometry>
-            <cylinder length="${wheel_len}" radius="${wheel_radius}"/>
+            <cylinder length="${wheel_width}" radius="${wheel_radius}"/>
           </geometry>
         </collision>
@@ -109,5 +114,5 @@
           <origin xyz="0 0 0" rpy="${PI/2} 0 ${PI/2}"/>
           <geometry>
-            <cylinder length="${wheel_len}" radius="${wheel_radius}"/>
+            <cylinder length="${wheel_width}" radius="${wheel_radius}"/>
           </geometry>
           <material name="black"/>
@@ -123,7 +128,7 @@
     </link>
     <joint name="${prefix}rear_left_wheel_joint" type="continuous">
-      <parent link="${prefix}chassis_link" />
+      <parent link="${prefix}base_link" />
       <child link="${prefix}rear_left_wheel" />
-      <origin xyz="-${wheelbase/2} -${base_width/2} -${base_height/2}" rpy="0 0 ${PI/2}"/>
+      <origin xyz="0 ${wheel_track/2} 0" rpy="0 0 ${PI/2}"/>
       <axis xyz="1 0 0"/>
       <limit effort="100.0" velocity="100.0"/>
@@ -143,7 +148,7 @@
     </link>
     <joint name="${prefix}virtual_front_wheel_joint" type="revolute">
-      <parent link="${prefix}chassis_link"/>
+      <parent link="${prefix}base_link"/>
       <child link="${prefix}virtual_front_wheel"/>
-      <origin xyz="${wheelbase/2} 0 -${base_height/2}" rpy="0 0 ${PI/2}"/>
+      <origin xyz="${wheel_base} 0 0" rpy="0 0 ${PI/2}"/>
       <axis xyz="0 0 1"/>
       <limit lower="-0.4" upper="0.4" effort="100.0" velocity="0.0"/>
@@ -155,5 +160,5 @@
         <origin xyz="0 0 0" rpy="${PI/2} 0 ${PI/2}"/>
         <geometry>
-          <cylinder length="${wheel_len}" radius="${wheel_radius}"/>
+          <cylinder length="${wheel_width}" radius="${wheel_radius}"/>
         </geometry>
       </collision>
@@ -161,5 +166,5 @@
         <origin xyz="0 0 0" rpy="${PI/2} 0 ${PI/2}"/>
         <geometry>
-          <cylinder length="${wheel_len}" radius="${wheel_radius}"/>
+          <cylinder length="${wheel_width}" radius="${wheel_radius}"/>
         </geometry>
         <material name="black"/>
@@ -175,7 +180,7 @@
     </link>
     <joint name="${prefix}front_right_wheel_joint" type="revolute">
-      <parent link="${prefix}chassis_link" />
+      <parent link="${prefix}base_link" />
       <child link="${prefix}front_right_wheel" />
-      <origin xyz="${wheelbase/2} ${base_width/2} -${base_height/2}" rpy="0 0 ${PI/2}"/>
+      <origin xyz="${wheel_base} -${wheel_track/2} 0" rpy="0 0 ${PI/2}"/>
       <axis xyz="0 0 1"/>
       <limit lower="-0.4" upper="0.4" effort="100.0" velocity="0.0"/>
@@ -188,5 +193,5 @@
         <origin xyz="0 0 0" rpy="${PI/2} 0 ${PI/2}"/>
         <geometry>
-          <cylinder length="${wheel_len}" radius="${wheel_radius}"/>
+          <cylinder length="${wheel_width}" radius="${wheel_radius}"/>
         </geometry>
       </collision>
@@ -194,5 +199,5 @@
         <origin xyz="0 0 0" rpy="${PI/2} 0 ${PI/2}"/>
         <geometry>
-          <cylinder length="${wheel_len}" radius="${wheel_radius}"/>
+          <cylinder length="${wheel_width}" radius="${wheel_radius}"/>
         </geometry>
         <material name="black"/>
@@ -208,7 +213,7 @@
     </link>
     <joint name="${prefix}front_left_wheel_joint" type="revolute">
-      <parent link="${prefix}chassis_link" />
+      <parent link="${prefix}base_link" />
       <child link="${prefix}front_left_wheel" />
-      <origin xyz="${wheelbase/2} -${base_width/2} -${base_height/2}" rpy="0 0 ${PI/2}"/>
+      <origin xyz="${wheel_base} ${wheel_track/2} 0" rpy="0 0 ${PI/2}"/>
       <axis xyz="0 0 1"/>
       <limit lower="-0.4" upper="0.4" effort="100.0" velocity="0.0"/>
